File: mcu.kicad_sch (KiCad schematic)
At the start: 16 parts, among them J1 Programming Connector, U1 PIC24FJ128GC010, Y1 48 MHz DNP

Commit message: Address review comments, finish routing HILT main board
Parts:
- removed R2, R3: 15R, Resistor_SMD:R_0805_2012Metric_Pad1.20x1.40mm_HandSolder, symbol Device:R_US
- C8, C9, Y1: now not fitted
Connections:
- net D+: now also U1.57 (D+/RG2)
- net D-: now also U1.56 (D-/RG3)
Other:
- note removed: "15R terminating resistors for USB."
- moved on the sheet: C7
Changed lines of the file:
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@@
-    (stroke (width 0) (type default))
-  )
-  (wire (pts (xy 88.9 55.88) (xy 91.44 55.88))
     (stroke (width 0) (type default))
   )
@@
     (stroke (width 0) (type default))
   )
-  (wire (pts (xy 88.9 58.42) (xy 91.44 58.42))
-    (stroke (width 0) (type default))
-  )
   (wire (pts (xy 44.45 46.99) (xy 39.37 46.99))
     (stroke (width 0) (type default))
@@
     (stroke (width 0) (type default))
   )
-  (wire (pts (xy 99.06 55.88) (xy 101.6 55.88))
-    (stroke (width 0) (type default))
-  )
   (wire (pts (xy 165.1 29.21) (xy 165.1 30.48))
     (stroke (width 0) (type default))
   )
-  (wire (pts (xy 86.36 53.34) (xy 86.36 50.8))
+  (wire (pts (xy 91.44 53.34) (xy 91.44 50.8))
     (stroke (width 0) (type default))
   )
@@
     (stroke (width 0) (type default))
   )
-  (wire (pts (xy 99.06 58.42) (xy 101.6 58.42))
-    (stroke (width 0) (type default))
-  )
-  (wire (pts (xy 101.6 53.34) (xy 86.36 53.34))
+  (wire (pts (xy 101.6 53.34) (xy 91.44 53.34))
     (stroke (width 0) (type default))
   )
@@
     (fill (type none))
   )
-  (text "15R terminating\nresistors for USB." (at 81.28 64.77 0)
-    (effects (font (size 1.27 1.27)) (justify left bottom))
-  )
   (text "AO pins are PPS remappable outputs which means they\ncan do PWM, and have associated analog input channels.\nAI1 - AI8 are PPS remappable inputs and have analog channels.\nAI9 - AI20 just have analog input channels.\nD1 - D2 have I2C support.\nD3 - D6 are PPS remappable inputs.\nD7 - D25 are regular digital I/O."
     (at 217.17 55.88 0)
@@
     (effects (font (size 1.27 1.27)) (justify left))
   )
-  (hierarchical_label "D-" (shape bidirectional) (at 88.9 58.42 180) (fields_autoplaced)
+  (hierarchical_label "D-" (shape bidirectional) (at 101.6 58.42 180) (fields_autoplaced)
     (effects (font (size 1.27 1.27)) (justify right))
   )
@@
     (effects (font (size 1.27 1.27)) (justify left))
   )
-  (hierarchical_label "D+" (shape bidirectional) (at 88.9 55.88 180) (fields_autoplaced)
+  (hierarchical_label "D+" (shape bidirectional) (at 101.6 55.88 180) (fields_autoplaced)
     (effects (font (size 1.27 1.27)) (justify right))
   )
@@
   (hierarchical_label "AI15" (shape bidirectional) (at 195.58 73.66 0) (fields_autoplaced)
     (effects (font (size 1.27 1.27)) (justify left))
-  )
-  (symbol (lib_id "Device:R_US") (at 95.25 58.42 90) (unit 1)
-    (in_bom yes) (on_board yes) (dnp no)
-    (property "Reference" "R3" (at 91.44 57.15 90)
-      (effects (font (size 1.27 1.27)))
-    )
-    (property "Value" "15R" (at 99.06 57.15 90)
-      (effects (font (size 1.27 1.27)))
-    )
-    (property "Footprint" "Resistor_SMD:R_0805_2012Metric_Pad1.20x1.40mm_HandSolder" (at 95.504 57.404 90)
-      (effects (font (size 1.27 1.27)) hide)
-    )
-    (property "Datasheet" "~" (at 95.25 58.42 0)
-      (effects (font (size 1.27 1.27)) hide)
-    )
-    (pin "1")
-    (pin "2")
-    (instances
-      (project "hil"
-        (path "/1993fdc2-1973-454b-bc68-679810c3998d"
-          (reference "R3") (unit 1)
-        )
-        (path "/1993fdc2-1973-454b-bc68-679810c3998d/62446467-ada0-4d3e-a3ad-0627169ed01a"
-          (reference "R5") (unit 1)
-        )
-      )
-    )
   )
   (symbol (lib_id "power:GND") (at 184.15 31.75 0) (unit 1)
@@
     )
   )
-  (symbol (lib_id "power:+3V3") (at 86.36 50.8 0) (unit 1)
+  (symbol (lib_id "power:+3V3") (at 91.44 50.8 0) (unit 1)
     (in_bom yes) (on_board yes) (dnp no) (fields_autoplaced)
-    (property "Reference" "#PWR011" (at 86.36 54.61 0)
-      (effects (font (size 1.27 1.27)) hide)
-    )
-    (property "Value" "+3V3" (at 86.36 47.2981 0)
-      (effects (font (size 1.27 1.27)))
-    )
-    (property "Footprint" "" (at 86.36 50.8 0)
-      (effects (font (size 1.27 1.27)) hide)
-    )
-    (property "Datasheet" "" (at 86.36 50.8 0)
+    (property "Reference" "#PWR011" (at 91.44 54.61 0)
+      (effects (font (size 1.27 1.27)) hide)
+    )
+    (property "Value" "+3V3" (at 91.44 47.2981 0)
+      (effects (font (size 1.27 1.27)))
+    )
+    (property "Footprint" "" (at 91.44 50.8 0)
+      (effects (font (size 1.27 1.27)) hide)
+    )
+    (property "Datasheet" "" (at 91.44 50.8 0)
       (effects (font (size 1.27 1.27)) hide)
     )
@@
     )
   )
-  (symbol (lib_id "power:+3V3") (at 76.2 50.8 0) (unit 1)
+  (symbol (lib_id "power:+3V3") (at 82.55 50.8 0) (unit 1)
     (in_bom yes) (on_board yes) (dnp no) (fields_autoplaced)
-    (property "Reference" "#PWR011" (at 76.2 54.61 0)
-      (effects (font (size 1.27 1.27)) hide)
-    )
-    (property "Value" "+3V3" (at 76.2 47.2981 0)
-      (effects (font (size 1.27 1.27)))
-    )
-    (property "Footprint" "" (at 76.2 50.8 0)
-      (effects (font (size 1.27 1.27)) hide)
-    )
-    (property "Datasheet" "" (at 76.2 50.8 0)
+    (property "Reference" "#PWR011" (at 82.55 54.61 0)
+      (effects (font (size 1.27 1.27)) hide)
+    )
+    (property "Value" "+3V3" (at 82.55 47.2981 0)
+      (effects (font (size 1.27 1.27)))
+    )
+    (property "Footprint" "" (at 82.55 50.8 0)
+      (effects (font (size 1.27 1.27)) hide)
+    )
+    (property "Datasheet" "" (at 82.55 50.8 0)
       (effects (font (size 1.27 1.27)) hide)
     )
@@
   )
   (symbol (lib_id "Device:C") (at 39.37 73.66 90) (unit 1)
-    (in_bom yes) (on_board yes) (dnp no) (fields_autoplaced)
+    (in_bom yes) (on_board yes) (dnp yes) (fields_autoplaced)
     (property "Reference" "C8" (at 39.37 68.4911 90)
       (effects (font (size 1.27 1.27)))
@@
   )
   (symbol (lib_id "Device:C") (at 39.37 86.36 90) (mirror x) (unit 1)
-    (in_bom yes) (on_board yes) (dnp no)
+    (in_bom yes) (on_board yes) (dnp yes)
     (property "Reference" "C9" (at 39.37 89.916 90)
       (effects (font (size 1.27 1.27)))
@@
   )
   (symbol (lib_id "Device:Crystal_GND24") (at 45.72 80.01 90) (unit 1)
-    (in_bom yes) (on_board yes) (dnp no)
+    (in_bom yes) (on_board yes) (dnp yes)
     (property "Reference" "Y1" (at 52.07 76.2 90)
       (effects (font (size 1.27 1.27)))
@@
         (path "/1993fdc2-1973-454b-bc68-679810c3998d/62446467-ada0-4d3e-a3ad-0627169ed01a"
           (reference "Y2") (unit 1)
-        )
-      )
-    )
-  )
-  (symbol (lib_id "Device:R_US") (at 95.25 55.88 90) (unit 1)
-    (in_bom yes) (on_board yes) (dnp no)
-    (property "Reference" "R2" (at 91.44 54.61 90)
-      (effects (font (size 1.27 1.27)))
-    )
-    (property "Value" "15R" (at 99.06 54.61 90)
-      (effects (font (size 1.27 1.27)))
-    )
-    (property "Footprint" "Resistor_SMD:R_0805_2012Metric_Pad1.20x1.40mm_HandSolder" (at 95.504 54.864 90)
-      (effects (font (size 1.27 1.27)) hide)
-    )
-    (property "Datasheet" "~" (at 95.25 55.88 0)
-      (effects (font (size 1.27 1.27)) hide)
-    )
-    (pin "1")
-    (pin "2")
-    (instances
-      (project "hil"
-        (path "/1993fdc2-1973-454b-bc68-679810c3998d"
-          (reference "R2") (unit 1)
-        )
-        (path "/1993fdc2-1973-454b-bc68-679810c3998d/62446467-ada0-4d3e-a3ad-0627169ed01a"
-          (reference "R4") (unit 1)
         )
       )
@@
     )
   )
-  (symbol (lib_id "power:GND") (at 76.2 58.42 0) (unit 1)
+  (symbol (lib_id "power:GND") (at 82.55 58.42 0) (unit 1)
     (in_bom yes) (on_board yes) (dnp no) (fields_autoplaced)
-    (property "Reference" "#PWR02" (at 76.2 64.77 0)
-      (effects (font (size 1.27 1.27)) hide)
-    )
-    (property "Value" "GND" (at 76.2 62.5555 0)
-      (effects (font (size 1.27 1.27)))
-    )
-    (property "Footprint" "" (at 76.2 58.42 0)
-      (effects (font (size 1.27 1.27)) hide)
-    )
-    (property "Datasheet" "" (at 76.2 58.42 0)
+    (property "Reference" "#PWR02" (at 82.55 64.77 0)
+      (effects (font (size 1.27 1.27)) hide)
+    )
+    (property "Value" "GND" (at 82.55 62.5555 0)
+      (effects (font (size 1.27 1.27)))
+    )
+    (property "Footprint" "" (at 82.55 58.42 0)
+      (effects (font (size 1.27 1.27)) hide)
+    )
+    (property "Datasheet" "" (at 82.55 58.42 0)
       (effects (font (size 1.27 1.27)) hide)
     )
@@
     )
   )
-  (symbol (lib_id "Device:C") (at 76.2 54.61 0) (unit 1)
+  (symbol (lib_id "Device:C") (at 82.55 54.61 0) (unit 1)
     (in_bom yes) (on_board yes) (dnp no)
-    (property "Reference" "C7" (at 76.2 52.07 0)
-      (effects (font (size 1.27 1.27)) (justify left))
-    )
-    (property "Value" "100n" (at 76.2 57.15 0)
-      (effects (font (size 1.27 1.27)) (justify left))
-    )
-    (property "Footprint" "Capacitor_SMD:C_0805_2012Metric_Pad1.18x1.45mm_HandSolder" (at 77.1652 58.42 0)
-      (effects (font (size 1.27 1.27)) hide)
-    )
-    (property "Datasheet" "~" (at 76.2 54.61 0)
-      (effects (font (size 1.27 1.27)) hide)
-    )
+    (property "Reference" "C7" (at 82.55 52.07 0)
+      (effects (font (size 1.27 1.27)) (justify left))
+    )
+    (property "Value" "100n" (at 82.55 57.15 0)
+      (effects (font (size 1.27 1.27)) (justify left))
+    )
+    (property "Footprint" "Capacitor_SMD:C_0805_2012Metric_Pad1.18x1.45mm_HandSolder" (at 83.5152 58.42 0)
+      (effects (font (size 1.27 1.27)) hide)
+    )
+    (property "Datasheet" "~" (at 82.55 54.61 0)
+      (effects (font (size 1.27 1.27)) hide)
+    )
